File: ST72F264 Programming Interface/ST72F264 Programming Interface.kicad_pcb (KiCad board)
At the start: 2 copper layers, 7 parts, among them J1 Conn_02x05_Odd_Even, U1 ST72F264, Y1 Resonator

Commit message: Board layout for production
Rev A of PCB layout
Parts:
- JP1, R1, TP1, TP2: moved to B.Cu
- moved JP1 217.4 mm to (131.0, 103.5), turned to 180 degrees
- moved J1 194.9 mm to (163.5, 107.5), turned to 90 degrees
- moved R1 192.9 mm to (140.0, 101.5), turned to 180 degrees
- moved TP2 191.7 mm to (135.5, 101.0)
- moved TP1 191.5 mm to (130.0, 101.0)
- moved U1 191.4 mm to (142.0, 102.1)
- moved Y1 191.4 mm to (131.2, 111.3)
Routing:
- net VDD: track 0.00 -> 58.0 mm
- net ~RESET: track 0.00 -> 41.3 mm
- net OSC: track 0.00 -> 41.2 mm
- net ICCSEL: track 0.00 -> 34.5 mm, vias 0 -> 1
- net ICCCLK: track 0.00 -> 32.8 mm, vias 0 -> 1
- net ICCDATA: track 0.00 -> 32.4 mm, vias 0 -> 1
- net Net-(JP1-Pad2): track 0.00 -> 8.55 mm
- net Net-(U1-Pad3): track 0.00 -> 4.72 mm
- net GND: track 0.00 -> 3.71 mm, vias 0 -> 5
- added copper zone on B.Cu, net GND
- added copper zone on F.Cu, net GND
Other:
- board outline added: 45.5 x 23 mm
- rule pad_to_mask_clearance: 0 -> 0.0508
- rule trace_min: 0.2 -> 0.1524
- rule via_min_drill: 0.3 -> 0.254
- rule via_min_size: 0.4 -> 0.38
